File: schematic ( kicad )/Nichel_H743/fc_nickel_v1.0.kicad_pcb (KiCad board)
At the start: 2 copper layers, 47 x 60 mm, 99 parts, among them J1 Micro_SD_Card_fc, J2 usb_typ_b_sym, Q1 SS8050, U1 STM32H743VITx, U2 SPX3819M5-L-3-3, U3 LM7805_TO220, U4 XC6504, U5 ICM42605, U6 ICM42688, U7 BMM150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

Commit message: updated unconnected crystal ground
updated unconnected crystal ground
Routing:
- net GND: track 482.4 -> 496.7 mm
- net /osc_1: track 28.7 -> 27.0 mm
- net /adc_v2: track 70.7 -> 72.2 mm
- net /osc_2: track 19.8 -> 19.1 mm
